File: TPA3128D2_GuitarAudioAmplifier_Mono/TPA3128D2_GuitarAudioAmplifier.kicad_pcb (KiCad board)
At the start: 2 copper layers, 55 x 30 mm, 30 parts, among them J1 SPEAKER, J2 INPUT, SW1 SW_SPDT, U1 TPA3128D2

Commit message: init
Parts:
- added G***: LOGO, LOGO, F.Cu at (128.6, 73.9)
Routing:
- net GND: vias 55 -> 53
